File: hardware/rev1.1/TangNanoDCJ11MEM.kicad_sch (KiCad schematic)
At the start: 38 parts, among them J1 Barrel_Jack_Switch, J2 VCC_FPGA, J3 CPU Vcc, J4 TangNano20K5VInterface, J5 Conn_01x20, J6 Conn_01x20, J7 UART, J8 Conn_01x30, J9 Conn_01x30, SW1 SW_SPDT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

Commit message: R2-6 changed
Parts:
- R2, R3, R4, R5, R6: value 100k -> 10k
Changed lines of the file:
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@@
 	(title_block
 		(title "Memory System and UART for DCJ11  using Tang Nano 20K")
-		(date "2024-04-24")
-		(rev "1.1")
+		(date "2024-07-15")
+		(rev "1.1a")
 		(company "Ryo Mukai")
+		(comment 1 "1.1 -> 1.1a: R2-R6 changed from 100k to 10k")
 	)
 	(junction
@@
 			)
 		)
-		(property "Value" "100k"
-			(at 171.45 151.13 90)
+		(property "Value" "10k"
+			(at 171.958 151.13 90)
 			(effects
 				(font
@@
 			)
 		)
-		(property "Value" "100k"
-			(at 171.45 148.59 90)
+		(property "Value" "10k"
+			(at 171.958 148.59 90)
 			(effects
 				(font
@@
 			)
 		)
-		(property "Value" "100k"
-			(at 171.45 146.05 90)
+		(property "Value" "10k"
+			(at 171.958 146.05 90)
 			(effects
 				(font
@@
 			)
 		)
-		(property "Value" "100k"
-			(at 163.83 132.08 90)
+		(property "Value" "10k"
+			(at 163.83 132.842 90)
 			(effects
 				(font
@@
 			)
 		)
-		(property "Value" "100k"
-			(at 171.45 153.67 90)
+		(property "Value" "10k"
+			(at 171.958 153.67 90)
 			(effects
 				(font
