File: hardware/rev2.1/TangNanoDCJ11MEM.kicad_pcb (KiCad board)
At the start: 2 copper layers, 99.1 x 99.1 mm, 36 parts, among them J1 TangNano20K5VInterface, J2 Conn_01x20, J3 Conn_01x20, J4 Conn_01x30, J5 Conn_01x30, J6 DBG UART, SW1 INIT, SW2 HALT, U1 DCJ11, Y1 18MHz

Commit message: PCB rev2.1 released
Parts:
- moved R15 19.2 mm to (69.8, 82.5), turned to 0 degrees
- moved SW2 2.54 mm to (81.3, 82.5)
Connections:
- J1 pad 16: HALT -> HALT_DBG
- J2 pad 16: HALT -> HALT_DBG
- R15 pad 1: Net-(R15-Pad1) -> HALT_DBG
- SW2 pad 2: Net-(R15-Pad1) -> HALT
Routing:
- net HALT_DBG: track 0.00 -> 29.2 mm, vias 0 -> 1
- net Net-(R15-Pad1): track 17.6 -> 0.00 mm
- net VCC: track 281.7 -> 278.5 mm
- net HALT: track 102.4 -> 102.1 mm, vias 3 -> 1
Other:
- board text added: "+5V"
- board text added: "[TN20KDCJ11MEM]rev.2.1"
- board text removed: "[TN20KDCJ11MEM]rev.2.0"
