File: hardware/rev2.1/TangNanoDCJ11MEM.kicad_sch (KiCad schematic)
At the start: 32 parts, among them J1 TangNano20K5VInterface, J2 Conn_01x20, J3 Conn_01x20, J4 Conn_01x30, J5 Conn_01x30, J6 DBG UART, SW1 INIT, SW2 HALT, U1 DCJ11, Y1 18MHz

Commit message: PCB rev2.1 released
Connections:
- net HALT: now also SW2.2; no longer J1.16 (Pin_16), J2.16 (Pin_16)
- net HALT_DBG: now reaches R15.1
- net HALT_DBG: now also J1.16 (Pin_16), J2.16 (Pin_16); no longer SW2.2
Other:
- note added: "resistor is for collision of HALT_SW and HALT_DBG"
- note removed: "to avoid collision with FPGA output"
- moved on the sheet: R15
Changed lines of the file:
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@@
 	(title_block
 		(title "Memory System and UART for DCJ11  using Tang Nano 20K")
-		(date "2025-08-26")
-		(rev "2.0")
+		(date "2025-09-05")
+		(rev "2.1")
 		(company "Ryo Mukai")
 		(comment 1 "modified to use CLK2")
+		(comment 2 "modified resisters of HALT and HALT_SW")
 	)
 	(junction
@@
 	)
 	(junction
+		(at 50.8 157.48)
+		(diameter 0)
+		(color 0 0 0 0)
+	)
+	(junction
 		(at 177.8 121.92)
 		(diameter 0)
@@
 	(wire
 		(pts
+			(xy 50.8 157.48) (xy 50.8 163.83)
+		)
+		(stroke
+			(width 0)
+			(type default)
+		)
+	)
+	(wire
+		(pts
 			(xy 45.72 157.48) (xy 50.8 157.48)
 		)
@@
 	(wire
 		(pts
+			(xy 50.8 157.48) (xy 58.42 157.48)
+		)
+		(stroke
+			(width 0)
+			(type default)
+		)
+	)
+	(wire
+		(pts
 			(xy 177.8 130.81) (xy 177.8 133.35)
 		)
@@
 	(wire
 		(pts
+			(xy 60.96 163.83) (xy 58.42 163.83)
+		)
+		(stroke
+			(width 0)
+			(type default)
+		)
+	)
+	(wire
+		(pts
 			(xy 170.18 156.21) (xy 165.1 156.21)
 		)
@@
 		)
 	)
-	(text "to avoid collision with\nFPGA output"
+	(text "resistor is for collision of\nHALT_SW and HALT_DBG"
 		(exclude_from_sim no)
-		(at 54.864 163.576 0)
+		(at 54.356 171.45 0)
 		(effects
 			(font
@@
 		)
 	)
-	(global_label "HALT"
+	(global_label "HALT_DBG"
+		(shape input)
+		(at 60.96 163.83 0)
+		(fields_autoplaced yes)
+		(effects
+			(font
+				(size 1.27 1.27)
+			)
+			(justify left)
+		)
+		(property "Intersheetrefs" "${INTERSHEET_REFS}"
+			(at 73.1376 163.83 0)
+			(effects
+				(font
+					(size 1.27 1.27)
+				)
+				(justify left)
+				(hide yes)
+			)
+		)
+	)
+	(global_label "HALT_DBG"
 		(shape input)
 		(at 129.54 71.12 180)
@@
 		)
 		(property "Intersheetrefs" "${INTERSHEET_REFS}"
-			(at 122.14 71.12 0)
+			(at 117.3624 71.12 0)
 			(effects
 				(font
@@
 		)
 	)
-	(global_label "HALT"
+	(global_label "HALT_DBG"
 		(shape input)
 		(at 63.5 71.12 180)
@@
 		)
 		(property "Intersheetrefs" "${INTERSHEET_REFS}"
-			(at 56.1 71.12 0)
+			(at 51.3224 71.12 0)
 			(effects
 				(font
@@
 	(symbol
 		(lib_id "000_MyLibrary:R")
-		(at 54.61 157.48 270)
+		(at 54.61 163.83 270)
 		(unit 1)
 		(exclude_from_sim no)
@@
 		(dnp no)
 		(property "Reference" "R15"
-			(at 53.34 160.274 90)
+			(at 53.34 166.624 90)
 			(effects
 				(font
@@
 		)
 		(property "Value" "1k"
-			(at 53.594 157.48 90)
+			(at 53.594 163.83 90)
 			(effects
 				(font
@@
 		)
 		(property "Footprint" "000_MyFootprint:R_Axial_DIN0207_L6.3mm_D2.5mm_P7.62mm_Horizontal"
-			(at 54.61 155.702 90)
+			(at 54.61 162.052 90)
 			(effects
 				(font
@@
 		)
 		(property "Datasheet" "~"
-			(at 54.61 157.48 0)
+			(at 54.61 163.83 0)
 			(effects
 				(font
@@
 		)
 		(property "Description" "Resistor"
-			(at 54.61 157.48 0)
+			(at 54.61 163.83 0)
 			(effects
 				(font
